File: RF1_12V/RF1_12V.sch (EAGLE design)
At the start: 17 parts, among them IC1 L78L33ACZ, IC2 MCP1702, J1 12V, Q1 16mhz, U1 ATMEGA328P_PDIP

Commit message: Updated with 2014 designs for both RF1_12v and RF1 5v
Parts:
- removed Q1: 16mhz, special:XTAL/S
- removed TP1: PTR1PAD1-13Y, testpad:PTR1PAD1-13Y
- added JP1: +12v, jumper:JP1E
- added U$2: (no value), adafruit:CERMOSCILL-THM
- C2: value .1uf -> .1uF
- C3, C4: value 1uF -> 10uF
- C5, C6: device resistor:C-EU025-024X044 -> adafruit:C-USC0805
- C7, C8: value 100n -> .1uF
- J1: device con-jack:DCJ0303 -> con-jack_komby:DCJ0303
Connections:
- net GND: now also U$2.GND
- net N$5: now also U$2.OUT; no longer Q1.2
- net N$6: now also U$2.IN; no longer Q1.1
- net VIN: now also JP1.1, JP1.2; no longer TP1.TP
Other:
- note added: "0.4"
- note removed: "0.1r1"
- moved on the sheet: C5, C6
